File: hardware/GeigerCounter/GeigerCounter.kicad_sch (KiCad schematic)
At the start: 20 parts, among them Q1 MMBTA44, Q2 MMBTA44, Q3 MMBT3904, U1 NE555D

Commit message: work with kicad
Parts:
- added J4: GameBoy_GamePak_DMG-09, SI3BG:Gameboy-Connector, symbol Connector_GameBoy:GameBoy_GamePak_DMG-09
- R6: footprint Resistor_SMD:R_0805_2012Metric_Pad1.20x1.40mm_HandSolder -> Resistor_SMD:R_2010_5025Metric_Pad1.40x2.65mm_HandSolder
Connections:
- net GND: now also J4.32 (GND)
- new net +5V: J4.1 (VCC)
- new net CARD_A0: J4.6 (A0)
- new net CARD_A1: J4.7 (A1)
- new net CARD_A10: J4.16 (A10)
- new net CARD_A11: J4.17 (A11)
- new net CARD_A12: J4.18 (A12)
- new net CARD_A13: J4.19 (A13)
- new net CARD_A14: J4.20 (A14), J4.31 (AUDIOIN)
- new net CARD_A15: J4.21 (A15)
- new net CARD_A2: J4.8 (A2)
- new net CARD_A3: J4.9 (A3)
- new net CARD_A4: J4.10 (A4)
- new net CARD_A5: J4.11 (A5)
- new net CARD_A6: J4.12 (A6)
- new net CARD_A7: J4.13 (A7)
- new net CARD_A8: J4.14 (A8)
- new net CARD_A9: J4.15 (A9)
- new net CARD_CLK: J4.2 (PHI)
- new net CARD_D0: J4.22 (D0)
- new net CARD_D1: J4.23 (D1)
- new net CARD_D2: J4.24 (D2)
- new net CARD_D3: J4.25 (D3)
- new net CARD_D4: J4.26 (D4)
- new net CARD_D5: J4.27 (D5)
- new net CARD_D6: J4.28 (D6)
- new net CARD_D7: J4.29 (D7)
- new net CARD_~{CS}: J4.5 (~{CS})
- new net CARD_~{RD}: J4.4 (~{RD})
- new net CARD_~{RES}: J4.30 (~{RST})
- new net CARD_~{WR}: J4.3 (~{WR})
- no-connect marks 1 -> 13
Other:
- note added: "D0-D7: data ADC6,ADC7: data WR|RD|CS|VIN: control CLK: button RES: reset <-> pull low VIN-A15: indicator"
- note added: "Vcc=5V!"

Commit message: work with kicad
Parts:
- R6: LCSC (none) -> C2765816
Changed lines of the file:
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@@
 			)
 		)
-		(property "Datasheet" "~"
+		(property "Datasheet" "https://www.lcsc.com/product-detail/C2765816.html"
 			(at 113.03 41.91 0)
 			(effects
@@
 			(effects
 				(font
+					(size 1.27 1.27)
+				)
+				(hide yes)
+			)
+		)
+		(property "LCSC" "C2765816"
+			(at 113.03 41.91 90)
+			(effects
+				(font

Commit message: change to 2 inductors
Parts:
- added L2: 4.7mH, EasyEDA:IND-SMD_L6.6-W4.4, symbol Device:L
- added TP1, TP2: TestPoint, Connector_PinSocket_2.54mm:PinSocket_1x01_P2.54mm_Vertical, symbol Connector:TestPoint
- L1: value 10mH -> 4.7mH; footprint Inductor_SMD:L_Bourns_SRR1208_12.7x12.7mm -> EasyEDA:IND-SMD_L6.6-W4.4; LCSC (none) -> C168108
Connections:
- net INT is gone; now on net CARD_D0: Q3.3 (C), R7.2
- net VCC is gone; now on net +5V: L1.1, R1.1, R7.1, U1.8 (VCC)
- net GND: now also TP2.1
- net at D2.2 (A), Q1.3 (C): now also L2.2, TP1.1; no longer L1.2
- new net: L1.2, L2.1
- no-connect marks 13 -> 22
Other:
- note added: "D0-D7: data ADC6,ADC7: data WR|RD|CS|VIN: control CLK: button RES: reset <-> pull low VIN-A14: indicator"
- note removed: "D0-D7: data ADC6,ADC7: data WR|RD|CS|VIN: control CLK: button RES: reset <-> pull low VIN-A15: indicator"
- moved on the sheet: L1, R1
